Commit message: Adjust launche files to standard name

File: src/Robot_5Dof_urdf/urdf/Robot_5Dof_gazebo.xacro (robot description, xacro)
@@ -3,6 +3,7 @@
     <!-- Define the ros_control plugin in Gazebo -->
     <gazebo>
-        <plugin name="control" filename="libgazebo_ros_control.so">
+        <plugin name="gazebo_ros_control" filename="libgazebo_ros_control.so">
             <robotNamespace>/</robotNamespace>
+            <robotSimType>gazebo_ros_control/DefaultRobotHWSim</robotSimType>
         </plugin>
     </gazebo>
@@ -10,16 +11,26 @@
     <gazebo reference="arm1_link">
         <selfCollide>true</selfCollide>
+        <material>Gazebo/Blue</material>
+        <gravity>true</gravity>
     </gazebo>
     <gazebo reference="arm2_link">
         <selfCollide>true</selfCollide>
+        <material>Gazebo/White</material>
+        <gravity>true</gravity>
     </gazebo>
     <gazebo reference="arm3_link">
         <selfCollide>true</selfCollide>
+        <material>Gazebo/Blue</material>
+        <gravity>true</gravity>
     </gazebo>
     <gazebo reference="arm4_link">
         <selfCollide>true</selfCollide>
+        <material>Gazebo/White</material>
+        <gravity>true</gravity>
     </gazebo>
     <gazebo reference="arm5_link">
         <selfCollide>true</selfCollide>
+        <material>Gazebo/Blue</material>
+        <gravity>true</gravity>
     </gazebo>
 </robot>

File: src/Robot_5Dof_urdf/urdf/Robot_5Dof_urdf.urdf.xacro (robot description, xacro)
@@ -3,5 +3,5 @@
      Commit Version: 1.6.0-1-g15f4949  Build Version: 1.6.7594.29634
      For more information, please see http://wiki.ros.org/sw_urdf_exporter -->
-<robot xmlns:xacro="http://www.ros.org/wiki/xacro" name="Robot_5Dof_urdf">
+<robot xmlns:xacro="http://www.ros.org/wiki/xacro" name="five_robot_arm">
   <!-- Define the world link -->
   <link name="world"/>
